File: PCB/Current/Skills.kicad_pcb (KiCad board)
At the start: 2 copper layers, 41 parts, among them U2 F-3188, U3 AP2112K-3.3

Commit message: working
Parts:
- added U5: TPS61088, Package_DFN_QFN:Texas_VQFN-RHL-20_ThermalVias, F.Cu at (160.0, 41.9)
Routing:
- added copper zone on B.Cu, net GND
Changed lines of the file:
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@@
     (tracks 0)
     (zones 0)
-    (modules 41)
-    (nets 80)
+    (modules 42)
+    (nets 83)
   )
   (page A4)
@@
   (net 78 "Net-(U2-Pad1)")
   (net 79 "Net-(U3-Pad4)")
+  (net 80 "Net-(U5-Pad11)")
+  (net 81 "Net-(U5-Pad12)")
+  (net 82 "Net-(U5-Pad13)")
   (net_class Default "This is the default net class."
     (clearance 0.2)
@@
     (add_net "Net-(U2-Pad43)")
     (add_net "Net-(U3-Pad4)")
+    (add_net "Net-(U5-Pad11)")
+    (add_net "Net-(U5-Pad12)")
+    (add_net "Net-(U5-Pad13)")
     (add_net SCK)
     (add_net SPI_EN)
+  )
+  (module Package_DFN_QFN:Texas_VQFN-RHL-20_ThermalVias (layer F.Cu)
+    (at 160.02 41.91)
+    (descr http://www.ti.com/lit/ds/symlink/bq51050b.pdf)
+    (tags RHL0020A)
+    (attr smd)
+    (fp_text reference U5 (at 0 -3.5) (layer F.SilkS)
+      (effects (font (size 1 1) (thickness 0.15)))
+    )
+    (fp_text value TPS61088 (at 0 3.7) (layer F.Fab)
+      (effects (font (size 1 1) (thickness 0.15)))
+    )
+    (fp_line (start -1.75 -1.73) (end -1.23 -2.25) (layer F.Fab) (width 0.1))
+    (fp_line (start -1.75 -1.73) (end -1.75 2.25) (layer F.Fab) (width 0.1))
+    (fp_line (start -1.75 2.25) (end 1.75 2.25) (layer F.Fab) (width 0.1))
+    (fp_line (start 1.75 -2.25) (end 1.75 2.25) (layer F.Fab) (width 0.1))
+    (fp_line (start -1.23 -2.25) (end 1.75 -2.25) (layer F.Fab) (width 0.1))
+    (fp_line (start -2.2 2.7) (end 2.2 2.7) (layer F.CrtYd) (width 0.05))
+    (fp_line (start 2.2 -2.7) (end 2.2 2.7) (layer F.CrtYd) (width 0.05))
+    (fp_line (start -2.2 -2.7) (end 2.2 -2.7) (layer F.CrtYd) (width 0.05))
+    (fp_line (start -2.2 -2.7) (end -2.2 2.7) (layer F.CrtYd) (width 0.05))
+    (fp_line (start 1 -2.3) (end 1.8 -2.3) (layer F.SilkS) (width 0.12))
+    (fp_line (start 1 2.3) (end 1.8 2.3) (layer F.SilkS) (width 0.12))
+    (fp_line (start 1.8 -2.3) (end 1.8 -2) (layer F.SilkS) (width 0.12))
+    (fp_line (start 1.8 2) (end 1.8 2.3) (layer F.SilkS) (width 0.12))
+    (fp_line (start -1.8 2.3) (end -1 2.3) (layer F.SilkS) (width 0.12))
+    (fp_line (start -1.8 2) (end -1.8 2.3) (layer F.SilkS) (width 0.12))
+    (fp_line (start -1.9 -2.3) (end -1 -2.3) (layer F.SilkS) (width 0.12))
+    (fp_text user %R (at 0 -3.5) (layer F.Fab)
+      (effects (font (size 1 1) (thickness 0.15)))
+    )
+    (pad 21 smd custom (at 0 0) (size 1.524 1.524) (layers F.Cu F.Mask)
+      (net 1 GND) (zone_connect 0)
+      (options (clearance outline) (anchor rect))
+      (primitives
+        (gr_poly (pts
+           (xy 1.025 1.525) (xy 1.025 -1.525) (xy 0.375 -1.525) (xy 0.375 -1.925) (xy -0.375 -1.925)
+           (xy -0.375 -1.525) (xy -1.025 -1.525) (xy -1.025 1.525) (xy -0.375 1.525) (xy -0.375 1.925)
+           (xy 0.375 1.925) (xy 0.375 1.525)) (width 0))
+      ))
+    (pad 1 smd roundrect (at -0.75 -2.15) (size 0.24 0.6) (layers F.Cu F.Paste F.Mask) (roundrect_rratio 0.21)
+      (net 34 "Net-(R11-Pad1)"))
+    (pad 2 smd roundrect (at -1.65 -1.75) (size 0.6 0.24) (layers F.Cu F.Paste F.Mask) (roundrect_rratio 0.21)
+      (net 2 +BATT))
+    (pad 3 smd roundrect (at -1.65 -1.25) (size 0.6 0.24) (layers F.Cu F.Paste F.Mask) (roundrect_rratio 0.21)
+      (net 33 "Net-(R10-Pad1)"))
+    (pad 4 smd roundrect (at -1.65 -0.75) (size 0.6 0.24) (layers F.Cu F.Paste F.Mask) (roundrect_rratio 0.21)
+      (net 3 "Net-(C16-Pad2)"))
+    (pad 5 smd roundrect (at -1.65 -0.25) (size 0.6 0.24) (layers F.Cu F.Paste F.Mask) (roundrect_rratio 0.21)
+      (net 3 "Net-(C16-Pad2)"))
+    (pad 6 smd roundrect (at -1.65 0.25) (size 0.6 0.24) (layers F.Cu F.Paste F.Mask) (roundrect_rratio 0.21)
+      (net 3 "Net-(C16-Pad2)"))
+    (pad 7 smd roundrect (at -1.65 0.75) (size 0.6 0.24) (layers F.Cu F.Paste F.Mask) (roundrect_rratio 0.21)
+      (net 3 "Net-(C16-Pad2)"))
+    (pad 8 smd roundrect (at -1.65 1.25) (size 0.6 0.24) (layers F.Cu F.Paste F.Mask) (roundrect_rratio 0.21)
+      (net 22 "Net-(C16-Pad1)"))
+    (pad 9 smd roundrect (at -1.65 1.75) (size 0.6 0.24) (layers F.Cu F.Paste F.Mask) (roundrect_rratio 0.21)
+      (net 2 +BATT))
+    (pad 10 smd roundrect (at -0.75 2.15) (size 0.24 0.6) (layers F.Cu F.Paste F.Mask) (roundrect_rratio 0.21)
+      (net 23 "Net-(C17-Pad1)"))
+    (pad 11 smd roundrect (at 0.75 2.15) (size 0.24 0.6) (layers F.Cu F.Paste F.Mask) (roundrect_rratio 0.21)
+      (net 80 "Net-(U5-Pad11)"))
+    (pad 12 smd roundrect (at 1.65 1.75) (size 0.6 0.24) (layers F.Cu F.Paste F.Mask) (roundrect_rratio 0.21)
+      (net 81 "Net-(U5-Pad12)"))
+    (pad 13 smd roundrect (at 1.65 1.25) (size 0.6 0.24) (layers F.Cu F.Paste F.Mask) (roundrect_rratio 0.21)
+      (net 82 "Net-(U5-Pad13)"))
+    (pad 14 smd roundrect (at 1.65 0.75) (size 0.6 0.24) (layers F.Cu F.Paste F.Mask) (roundrect_rratio 0.21)
+      (net 6 +12V))
+    (pad 15 smd roundrect (at 1.65 0.25) (size 0.6 0.24) (layers F.Cu F.Paste F.Mask) (roundrect_rratio 0.21)
+      (net 6 +12V))
+    (pad 16 smd roundrect (at 1.65 -0.25) (size 0.6 0.24) (layers F.Cu F.Paste F.Mask) (roundrect_rratio 0.21)
+      (net 6 +12V))
+    (pad 17 smd roundrect (at 1.65 -0.75) (size 0.6 0.24) (layers F.Cu F.Paste F.Mask) (roundrect_rratio 0.21)
+      (net 39 "Net-(R16-Pad2)"))
+    (pad 18 smd roundrect (at 1.65 -1.25) (size 0.6 0.24) (layers F.Cu F.Paste F.Mask) (roundrect_rratio 0.21)
+      (net 36 "Net-(R13-Pad2)"))
+    (pad 19 smd roundrect (at 1.65 -1.75) (size 0.6 0.24) (layers F.Cu F.Paste F.Mask) (roundrect_rratio 0.21)
+      (net 37 "Net-(R14-Pad1)"))
+    (pad 20 smd roundrect (at 0.75 -2.15) (size 0.24 0.6) (layers F.Cu F.Paste F.Mask) (roundrect_rratio 0.21)
+      (net 1 GND))
+    (pad 21 smd roundrect (at -0.275 -2.15) (size 0.2 0.6) (layers F.Cu F.Paste F.Mask) (roundrect_rratio 0.25)
+      (net 1 GND))
+    (pad 21 smd roundrect (at 0.275 -2.15) (size 0.2 0.6) (layers F.Cu F.Paste F.Mask) (roundrect_rratio 0.25)
+      (net 1 GND))
+    (pad 21 smd roundrect (at -0.275 2.15) (size 0.2 0.6) (layers F.Cu F.Paste F.Mask) (roundrect_rratio 0.25)
+      (net 1 GND))
+    (pad 21 smd roundrect (at 0.275 2.15) (size 0.2 0.6) (layers F.Cu F.Paste F.Mask) (roundrect_rratio 0.25)
+      (net 1 GND))
+    (pad 21 thru_hole circle (at 0 0.525) (size 0.5 0.5) (drill 0.2) (layers *.Cu)
+      (net 1 GND) (zone_connect 2))
+    (pad 21 thru_hole circle (at 0 -0.525) (size 0.5 0.5) (drill 0.2) (layers *.Cu)
+      (net 1 GND) (zone_connect 2))
+    (pad 21 thru_hole circle (at -0.775 -0.525) (size 0.5 0.5) (drill 0.2) (layers *.Cu)
+      (net 1 GND) (zone_connect 2))
+    (pad 21 thru_hole circle (at 0.775 -0.525) (size 0.5 0.5) (drill 0.2) (layers *.Cu)
+      (net 1 GND) (zone_connect 2))
+    (pad 21 thru_hole circle (at -0.775 0.525) (size 0.5 0.5) (drill 0.2) (layers *.Cu)
+      (net 1 GND) (zone_connect 2))
+    (pad 21 thru_hole circle (at 0.775 0.525) (size 0.5 0.5) (drill 0.2) (layers *.Cu)
+      (net 1 GND) (zone_connect 2))
+    (pad 21 thru_hole circle (at 0 -1.275) (size 0.5 0.5) (drill 0.2) (layers *.Cu)
+      (net 1 GND) (zone_connect 2))
+    (pad 21 thru_hole circle (at 0 1.275) (size 0.5 0.5) (drill 0.2) (layers *.Cu)
+      (net 1 GND) (zone_connect 2))
+    (pad "" smd rect (at -0.56 -1.05) (size 0.92 0.85) (layers F.Paste))
+    (pad "" smd rect (at 0.56 -1.05) (size 0.92 0.85) (layers F.Paste))
+    (pad "" smd rect (at -0.56 0) (size 0.92 0.85) (layers F.Paste))
+    (pad "" smd rect (at 0.56 0) (size 0.92 0.85) (layers F.Paste))
+    (pad "" smd rect (at -0.56 1.05) (size 0.92 0.85) (layers F.Paste))
+    (pad "" smd rect (at 0.56 1.05) (size 0.92 0.85) (layers F.Paste))
+    (pad "" smd rect (at 0 -1.8) (size 0.75 0.25) (layers F.Paste))
+    (pad "" smd rect (at 0 1.8) (size 0.75 0.25) (layers F.Paste))
+    (model ${KISYS3DMOD}/Package_DFN_QFN.3dshapes/Texas_VQFN-RHL-20_ThermalVias.wrl
+      (at (xyz 0 0 0))
+      (scale (xyz 1 1 1))
+      (rotate (xyz 0 0 0))
+    )
   )
   (module Package_TO_SOT_SMD:SOT-23-5 (layer F.Cu)
@@
     )
   )
+  (zone (net 1) (net_name GND) (layer B.Cu) (hatch edge 0.508)
+    (connect_pads (clearance 0.508))
+    (min_thickness 0.254)
+    (fill yes (arc_segments 32) (thermal_gap 0.508) (thermal_bridge_width 0.508))
+    (polygon
+      (pts
+        (xy 155.448 36.83) (xy 167.894 36.068) (xy 170.18 45.974) (xy 158.496 52.07) (xy 144.272 48.514)
+        (xy 141.478 35.052)
+      )
+    )
+  )
