File: PCB/Current/Skills.kicad_pcb (KiCad board)
At the start: 2 copper layers, 70 x 85 mm, 71 parts, among them J1 USB_C_Receptacle_USB2.0, J2 BATT, J3 L, J4 SPI, J5 R, U1 TPS61088, U2 TP4056, U3 FS312F, U4 FS8205A, U5 ME6209, U6 F-3188, U7 MAX9744

Commit message: work in progress
Parts:
- removed the C1 at (84.3, 104.1)
- removed C22: 100n, Capacitor_SMD:C_0603_1608Metric
- removed C24: 2.2u, Capacitor_SMD:C_0603_1608Metric
- removed the J4 at (57.3, 99.1)
- removed the JP1 at (57.3, 80.5)
- removed L1: 1.5u, Inductor_SMD:L_Wuerth_HCI-1040
- removed L2: L, Inductor_SMD:L_0805_2012Metric
- removed the R11 at (107.8, 130.2)
- removed R16, R19, R20: 10k, Resistor_SMD:R_0603_1608Metric
- removed R17, R18: 1k, Resistor_SMD:R_0603_1608Metric
- removed the R2 at (76.3, 112.0)
- removed the R3 at (84.7, 115.2)
- removed the R5 at (76.3, 115.2)
- removed the R6 at (79.6, 115.2)
- removed REF**: KiCad-Logo2_5mm_SilkScreen, Symbol:KiCad-Logo2_5mm_SilkScreen
- removed the U1 at (82.0, 109.6)
- removed the U5 at (97.9, 75.2)
- removed U7: MAX9744, Package_DFN_QFN:QFN-44-1EP_7x7mm_P0.5mm_EP5.15x5.15mm_ThermalVias
- added J1: SPI, Connector_Molex:Molex_KK-254_AE-6410-05A_1x05_P2.54mm_Vertical, F.Cu at (64.3, 92.4)
- added JP2: AGND, Connector_PinHeader_2.54mm:PinHeader_1x02_P2.54mm_Vertical, F.Cu at (64.3, 98.6)
- added JP3: Jumper_NC_Dual, Jumper:SolderJumper-3_P1.3mm_Open_RoundedPad1.0x1.5mm_NumberLabels, F.Cu at (79.5, 90.2)
- added JP4: Jumper_NC_Dual, Jumper:SolderJumper-3_P1.3mm_Open_RoundedPad1.0x1.5mm_NumberLabels, F.Cu at (69.4, 98.0)
- added R1: 1k, Resistor_SMD:R_0603_1608Metric, F.Cu at (90.3, 97.2)
- added R13: 1k, Resistor_SMD:R_0603_1608Metric, F.Cu at (88.7, 102.2)
- added R7: 10k, Resistor_SMD:R_0603_1608Metric, F.Cu at (90.5, 82.2)
- added RV2: R_POT, Potentiometer_THT:Potentiometer_Bourns_3296W_Vertical, F.Cu at (99.0, 57.2)
- added RV3: R_POT, Potentiometer_THT:Potentiometer_Bourns_3296W_Vertical, F.Cu at (99.0, 63.6)
- added U2: TPA6132A2RTE, Package_DFN_QFN:WQFN-16-1EP_3x3mm_P0.5mm_EP1.6x1.6mm_ThermalVias, F.Cu at (79.4, 94.6)
- added U3: PAM8403, Package_SO:SOIC-16_3.9x9.9mm_P1.27mm, F.Cu at (82.5, 79.7)
- C1: renamed from C23; value 100n -> 100u
- C10: value 1n -> 1uF
- C11, C15, C16: value 10u -> 1uF; footprint Capacitor_SMD:C_0805_2012Metric -> Capacitor_SMD:C_0603_1608Metric
- C12: value 100n -> 100uF
- C13, C14: value 10u -> 470nF; footprint Capacitor_SMD:C_0805_2012Metric -> Capacitor_SMD:C_0603_1608Metric
- C17: value 470n -> 1uF
- C18, C20, C21: value 100n -> 1uF
- C19: value 470n -> 100uF
- C2, C3: value 10u -> 470nF; footprint Capacitor_SMD:C_1206_3216Metric -> Capacitor_SMD:C_0603_1608Metric
- C4, C5: value 22u -> 470nF; footprint Capacitor_SMD:C_1206_3216Metric -> Capacitor_SMD:C_0603_1608Metric
- C6: value 22u -> 1uF; footprint Capacitor_SMD:C_1206_3216Metric -> Capacitor_SMD:C_0603_1608Metric
- C7: value 100u -> 1uF; footprint Capacitor_SMD:CP_Elec_6.3x7.7 -> Capacitor_SMD:C_0603_1608Metric
- C8: value 2.2u -> 1uF
- C9: value 47n -> 1uF
- J2: renamed from J3; footprint Molex:Molex 2Pin -> Connector_Molex:Molex_KK-254_AE-6410-02A_1x02_P2.54mm_Vertical
- J3: renamed from J5; footprint Molex:Molex 2Pin -> Connector_Molex:Molex_KK-254_AE-6410-02A_1x02_P2.54mm_Vertical
- J5: renamed from J2; footprint Molex:Molex 3Pin -> Connector_Molex:Molex_KK-254_AE-6410-03A_1x03_P2.54mm_Vertical
- R15: value 10k -> 1k
- R4: value 44.2k -> 1k
- R5: renamed from R22; value 10k -> 1k
- R8: value 1.1k -> 10k
- moved R12 51.9 mm to (88.7, 99.7)
- moved R8 42.4 mm to (90.5, 84.7), turned to 0 degrees
- moved C11 41.3 mm to (88.4, 89.7), turned to 0 degrees
- moved C12 38.6 mm to (76.6, 101.0), turned to 0 degrees
- moved C20 30.5 mm to (80.6, 103.5), turned to 0 degrees
- moved C3 29.9 mm to (68.6, 103.6), turned to 0 degrees
- moved C14 26.7 mm to (82.3, 98.5)
- moved C10 23.9 mm to (84.4, 92.2), turned to 0 degrees
- moved C15 22.7 mm to (76.6, 103.5), turned to 0 degrees
- moved C21 22.1 mm to (84.7, 101.0), turned to 0 degrees
- moved C18 21.1 mm to (88.0, 94.7), turned to 0 degrees
- moved C17 20.5 mm to (72.6, 101.1), turned to 0 degrees
- moved R15 20.3 mm to (88.7, 104.7), turned to 0 degrees
- moved C4 19.4 mm to (84.4, 89.7), turned to 0 degrees
- moved C2 19.3 mm to (80.6, 101.0), turned to 0 degrees
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- renumbered D4 to D1, D5 to D2, D6 to D3, D1 to D4, D2 to D5, D3 to D6, J1 to J4, JP2 to JP1, R9 to R10, R10 to R11, R7 to R14, R13 to R2, R14 to R3, R21 to R6, R1 to R9, U6 to U1, U2 to U4, U3 to U5, U4 to U6
Connections:
- C1 pad 1: Net-(C23-Pad1) -> Net-(C1-Pad1)
- C10 pad 1: Net-(C10-Pad1) -> +BATT
- C11 pad 1: VBUS -> +BATT
- C12 pad 1: Net-(C12-Pad1) -> +BATT
- C12 pad 2: Net-(C12-Pad2) -> GND
- C13 pad 1: +12V -> Net-(C13-Pad1)
- C13 pad 2: GND -> Net-(C13-Pad2)
- C14 pad 1: +12V -> Net-(C14-Pad1)
- C14 pad 2: GND -> Net-(C14-Pad2)
- C15 pad 1: +3V3 -> Net-(C15-Pad1)
- C16 pad 1: +3V3 -> +BATT
- C17 pad 1: Net-(C17-Pad1) -> +BATT
- C17 pad 2: Net-(C17-Pad2) -> GND
- C18 pad 1: Net-(C18-Pad1) -> +BATT
- C18 pad 2: Net-(C18-Pad2) -> GND
- C19 pad 1: Net-(C19-Pad1) -> +BATT
- C19 pad 2: Net-(C17-Pad2) -> GND
- C2 pad 1: +BATT -> Net-(C2-Pad1)
- C2 pad 2: GND -> Net-(C2-Pad2)
- C20 pad 1: Net-(C20-Pad1) -> VBUS
- C20 pad 2: Net-(C20-Pad2) -> GND
- C3 pad 1: +BATT -> Net-(C3-Pad1)
- C3 pad 2: GND -> Net-(C3-Pad2)
- C5 pad 1: Net-(C4-Pad1) -> Net-(C5-Pad1)
- C6 pad 1: +12V -> Net-(C6-Pad1)
- C7 pad 1: +12V -> +BATT
- C8 pad 2: GND -> Net-(C8-Pad2)
- C9 pad 1: Net-(C9-Pad1) -> +BATT
- D1 pad 1: Net-(D4-Pad1) -> Net-(D1-Pad1)
- J2 pad 1: Net-(C20-Pad1) -> Net-(J2-Pad1)
- J2 pad 2: Net-(C18-Pad1) -> Net-(J2-Pad2)
- J3 pad 1: Net-(C21-Pad1) -> Net-(J3-Pad1)
- J5 pad 3: Net-(C12-Pad2) -> Net-(C21-Pad2)
- R12 pad 1: Net-(D4-Pad1) -> Net-(R12-Pad1)
- R14 pad 1: Net-(C12-Pad1) -> Net-(C21-Pad1)
- R15 pad 2: Net-(C17-Pad1) -> GND
- R4 pad 1: Net-(R4-Pad1) -> Net-(C1-Pad1)
- R4 pad 2: Net-(C10-Pad1) -> GND
- R5 pad 2: Net-(C23-Pad1) -> Net-(C1-Pad1)
- R8 pad 1: Net-(R8-Pad1) -> Net-(C14-Pad1)
- R8 pad 2: GND -> Net-(R8-Pad2)
- RV1 pad 1: GND -> Net-(RV1-Pad1)
- RV1 pad 3: Net-(RV1-Pad3) -> GND
- U1 pad 15: Net-(C23-Pad1) -> Net-(C1-Pad1)
- U1 pad 3: Net-(R12-Pad2) -> Net-(R1-Pad2)
- U1 pad 39: Net-(U6-Pad39) -> Net-(C3-Pad2)
- U1 pad 40: Net-(R18-Pad2) -> Net-(C2-Pad2)
- U4 pad 2: Net-(R8-Pad1) -> Net-(R12-Pad1)
- U5 pad 2: Net-(R11-Pad1) -> Net-(R15-Pad1)
- U5 pad 5: Net-(C12-Pad1) -> Net-(C21-Pad1)
- U5 pad 6: Net-(C12-Pad2) -> Net-(C21-Pad2)
- U6 pad 2: Net-(C12-Pad2) -> Net-(C21-Pad2)
- U6 pad 3: Net-(C12-Pad2) -> Net-(C21-Pad2)
Routing:
- net +BATT: track 183.2 -> 0.00 mm, vias 2 -> 0
- net +12V: track 109.0 -> 0.00 mm
- net Net-(F1-Pad1): track 106.4 -> 0.00 mm, vias 1 -> 0
- net GND: track 74.2 -> 0.00 mm, vias 347 -> 0
- net Net-(RV1-Pad3): track 53.6 -> 0.00 mm, vias 2 -> 0
- net MISO: track 47.6 -> 0.00 mm
- net CSB: track 43.8 -> 0.00 mm
- net +3V3: track 40.4 -> 0.00 mm
- net Net-(C17-Pad2): track 40.3 -> 0.00 mm
- net CLK: track 40.1 -> 0.00 mm
- net Net-(RV1-Pad2): track 39.9 -> 0.00 mm, vias 2 -> 0
- net MOSI: track 36.3 -> 0.00 mm
- net VBUS: track 32.4 -> 0.00 mm
- net Net-(C12-Pad2): track 29.6 -> 0.00 mm
- net Net-(C18-Pad1): track 17.1 -> 0.00 mm
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- removed copper zone on F.Cu, net +BATT
- removed copper zone on F.Cu, net Net-(C1-Pad2)
- removed copper zone on F.Cu, net Net-(C4-Pad1)

Commit message: work in progress
Parts:
- removed D3: LED, LED_SMD:LED_0603_1608Metric
- removed R3: 1k, Resistor_SMD:R_0603_1608Metric
- added JP5: LEDs, Connector_PinHeader_2.54mm:PinHeader_1x02_P2.54mm_Vertical, F.Cu at (86.6, 96.4)
- added JP8: Jumper_NC_Dual, Connector_PinHeader_2.54mm:PinHeader_1x03_P2.54mm_Vertical, F.Cu at (82.0, 96.4)
- J1: footprint Connector_Molex:Molex_KK-254_AE-6410-05A_1x05_P2.54mm_Vertical -> Connector_PinHeader_2.54mm:PinHeader_1x05_P2.54mm_Vertical
- JP3, JP4: footprint Jumper:SolderJumper-3_P1.3mm_Open_RoundedPad1.0x1.5mm_NumberLabels -> Connector_PinHeader_2.54mm:PinHeader_1x03_P2.54mm_Vertical
- moved RV3 60.1 mm to (63.6, 112.1)
- moved RV2 46.0 mm to (76.7, 97.3)
- moved U3 27.2 mm to (64.3, 99.8)
- moved C3 26.5 mm to (95.0, 100.4)
- moved R8 25.5 mm to (87.8, 110.1)
- moved C14 21.8 mm to (62.1, 106.8)
- moved C4 20.4 mm to (83.8, 110.1)
- moved U2 19.1 mm to (73.9, 112.9)
- moved C11 17.9 mm to (87.8, 107.6)
- moved C5 17.2 mm to (78.5, 115.1)
- moved C6 16.6 mm to (78.5, 112.6)
- moved R7 16.3 mm to (95.0, 97.9)
- moved C13 16.0 mm to (79.8, 110.1)
- moved C17 15.7 mm to (87.8, 105.1)
- moved JP3 15.4 mm to (70.9, 102.9)
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Connections:
- D1 pad 2: +BATT -> Net-(D1-Pad2)
- D2 pad 2: +BATT -> Net-(D1-Pad2)
- D4 pad 1: GND -> Net-(D4-Pad1)
- U1 pad 1: Net-(R3-Pad2) -> LED
Other:
- board text removed: "Damian Stefan Lorenz"

Commit message: work in progress
Parts:
- removed the C3 at (95.0, 100.4)
- removed the J1 at (57.8, 96.4)
- removed JP8: Jumper_NC_Dual, Connector_PinHeader_2.54mm:PinHeader_1x03_P2.54mm_Vertical
- removed the R1 at (91.8, 107.9)
- removed the R12 at (91.8, 105.4)
- removed R15: 1k, Resistor_SMD:R_0603_1608Metric
- removed the R7 at (95.0, 97.9)
- removed the U2 at (73.9, 112.9)
- removed the U3 at (64.3, 99.8)
- added C1: 1uF, Capacitor_SMD:C_0603_1608Metric, F.Cu at (87.1, 96.3)
- added C22: 1uF, Capacitor_SMD:C_0603_1608Metric, F.Cu at (87.3, 108.9)
- added C23: 100uF, Capacitor_SMD:C_0603_1608Metric, F.Cu at (92.6, 101.7)
- added J3: SPI, Connector_PinHeader_2.54mm:PinHeader_1x05_P2.54mm_Vertical, F.Cu at (51.8, 82.3)
- added JP6: Jumper_NC_Dual, Connector_PinHeader_2.54mm:PinHeader_1x03_P2.54mm_Vertical, F.Cu at (82.7, 90.2)
- added R11: 1k, Resistor_SMD:R_0603_1608Metric, F.Cu at (83.3, 106.4)
- added R14: 10k, Resistor_SMD:R_0603_1608Metric, F.Cu at (88.6, 99.2)
- added R3: 1k, Resistor_SMD:R_0603_1608Metric, F.Cu at (87.3, 106.4)
- added R6: 1k, Resistor_SMD:R_0603_1608Metric, F.Cu at (95.1, 96.7)
- added U5: TPA6132A2RTE, Package_DFN_QFN:WQFN-16-1EP_3x3mm_P0.5mm_EP1.6x1.6mm_ThermalVias, F.Cu at (74.6, 106.7)
- added U6: PAM8403, Package_SO:SOIC-16_3.9x9.9mm_P1.27mm, F.Cu at (97.0, 77.8)
- C12, C19: value 100uF -> 1uF
- C13, C14, C2, C4: value 470nF -> 1uF
- C15: value 1uF -> 100uF
- C17, C18, C6, C7, C8, C9: value 1uF -> 470nF
- C5: value 470nF -> 100uF
- JP2: value AGND -> Jumper_NC_Dual; footprint Connector_PinHeader_2.54mm:PinHeader_1x02_P2.54mm_Vertical -> Connector_PinHeader_2.54mm:PinHeader_1x03_P2.54mm_Vertical
- JP3: value Jumper_NC_Dual -> LEDs; footprint Connector_PinHeader_2.54mm:PinHeader_1x03_P2.54mm_Vertical -> Connector_PinHeader_2.54mm:PinHeader_1x02_P2.54mm_Vertical
- JP4: value Jumper_NC_Dual -> AGND; footprint Connector_PinHeader_2.54mm:PinHeader_1x03_P2.54mm_Vertical -> Connector_PinHeader_2.54mm:PinHeader_1x02_P2.54mm_Vertical
- JP5: value LEDs -> Jumper_NC_Dual; footprint Connector_PinHeader_2.54mm:PinHeader_1x02_P2.54mm_Vertical -> Connector_PinHeader_2.54mm:PinHeader_1x03_P2.54mm_Vertical
- R13: value 1k -> 10k
- R8: value 10k -> 1k
- moved RV3 61.3 mm to (101.5, 64.0)
- moved RV2 48.0 mm to (101.6, 56.3)
- moved C14 33.3 mm to (91.7, 91.6)
- moved C8 24.7 mm to (66.8, 100.6)
- moved R4 22.9 mm to (95.7, 91.6)
- moved C15 21.4 mm to (62.8, 100.6)
- moved C9 18.4 mm to (62.2, 110.4)
- moved JP4 17.4 mm to (87.4, 90.2)
- moved JP2 16.1 mm to (71.6, 96.6)
- moved C18 15.6 mm to (91.7, 94.1)
- moved C4 15.3 mm to (91.1, 96.7)
- moved C10 14.5 mm to (91.7, 89.1)
- moved R13 12.5 mm to (88.6, 101.7)
- moved C16 12.2 mm to (95.7, 89.1)
- moved C19 12.0 mm to (84.6, 101.3)
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- renumbered C1 to C3, D5 to D1, D6 to D2, D4 to D3, D1 to D4, D2 to D5, J4 to J1, J5 to J2, J2 to J4, J3 to J5, R10 to R1, R9 to R10, R2 to R12, R11 to R2, R14 to R5, R6 to R7, R5 to R9, U4 to U1, U5 to U2, U6 to U3, U1 to U4
Connections:
- C10 pad 1: +BATT -> Net-(C10-Pad1)
- C13 pad 1: Net-(C13-Pad1) -> +BATT
- C13 pad 2: Net-(C13-Pad2) -> GND
- C14 pad 1: Net-(C14-Pad1) -> +BATT
- C14 pad 2: Net-(C14-Pad2) -> GND
- C15 pad 1: Net-(C15-Pad1) -> +BATT
- C16 pad 1: +BATT -> Net-(C16-Pad1)
- C16 pad 2: GND -> Net-(C16-Pad2)
- C17 pad 1: +BATT -> Net-(C17-Pad1)
- C17 pad 2: GND -> Net-(C17-Pad2)
- C18 pad 1: +BATT -> Net-(C18-Pad1)
- C18 pad 2: GND -> Net-(C18-Pad2)
- C19 pad 1: +BATT -> Net-(C19-Pad1)
- C20 pad 1: VBUS -> +BATT
- C21 pad 1: Net-(C21-Pad1) -> +BATT
- C21 pad 2: Net-(C21-Pad2) -> GND
- C3 pad 1: Net-(C1-Pad1) -> Net-(C3-Pad1)
- C4 pad 1: Net-(C4-Pad1) -> +BATT
- C5 pad 1: Net-(C5-Pad1) -> +BATT
- C6 pad 2: GND -> Net-(C6-Pad2)
- C7 pad 1: +BATT -> Net-(C7-Pad1)
- C7 pad 2: GND -> Net-(C7-Pad2)
- C8 pad 2: Net-(C8-Pad2) -> GND
- C9 pad 1: +BATT -> Net-(C9-Pad1)
- D3 pad 1: Net-(D4-Pad1) (its old number) -> Net-(D3-Pad1)
- D4 pad 2: Net-(D1-Pad2) -> Net-(D4-Pad2)
- D5 pad 2: Net-(D1-Pad2) -> Net-(D4-Pad2)
- J2 pad 3: Net-(C21-Pad2) -> Net-(C2-Pad2)
- JP2 pad 2: Net-(JP2-Pad2) -> Net-(D3-Pad1)
- JP3 pad 1: GND -> Net-(D4-Pad2)
- JP3 pad 2: Net-(JP3-Pad2) -> +BATT
- JP5 pad 1: Net-(D1-Pad2) -> GND
- JP5 pad 2: +BATT -> Net-(JP5-Pad2)
- R13 pad 2: GND -> Net-(C17-Pad1)
- R4 pad 1: Net-(C1-Pad1) -> Net-(R3-Pad2)
- R5 pad 1: Net-(C21-Pad1) -> Net-(C2-Pad1)
- R8 pad 1: Net-(C14-Pad1) -> Net-(C3-Pad1)
- R8 pad 2: Net-(R8-Pad2) -> GND
- R9 pad 2: Net-(C1-Pad1) -> Net-(C3-Pad1)
- RV2 pad 2: Net-(C13-Pad2) -> Net-(C17-Pad2)
- RV3 pad 2: Net-(C14-Pad2) -> Net-(C18-Pad2)
- U2 pad 5: Net-(C21-Pad1) -> Net-(C2-Pad1)
- U2 pad 6: Net-(C21-Pad2) -> Net-(C2-Pad2)
- U3 pad 2: Net-(C21-Pad2) -> Net-(C2-Pad2)
- U3 pad 3: Net-(C21-Pad2) -> Net-(C2-Pad2)
- U4 pad 15: Net-(C1-Pad1) -> Net-(C3-Pad1)
- U4 pad 39: Net-(C3-Pad2) -> Net-(C7-Pad2)
- U4 pad 40: Net-(C2-Pad2) -> Net-(C6-Pad2)
- U4 pad 43: Net-(JP2-Pad2) -> Net-(JP4-Pad2)

Commit message: work in progress
Parts:
- added C24: 1uF, Capacitor_SMD:C_0603_1608Metric, F.Cu at (87.8, 88.1)
- added JP7: Jumper_NC_Dual, Connector_PinHeader_2.54mm:PinHeader_1x03_P2.54mm_Vertical, F.Cu at (83.1, 78.0)
- added U7: CAT809, Package_TO_SOT_SMD:SOT-23, F.Cu at (83.5, 89.2)
- C15, C23, C3, C5: footprint Capacitor_SMD:C_0603_1608Metric -> Capacitor_SMD:CP_Elec_6.3x7.7
- moved C7 49.4 mm to (70.4, 62.5)
- moved C9 44.1 mm to (70.4, 67.1)
- moved C6 43.3 mm to (70.4, 64.0)
- moved R8 43.1 mm to (51.8, 113.0)
- moved D5 42.8 mm to (63.5, 99.8)
- moved R12 42.8 mm to (66.7, 99.8)
- moved D4 42.8 mm to (63.5, 101.5)
- moved U5 42.7 mm to (66.4, 64.8), turned to 180 degrees
- moved C12 40.2 mm to (64.6, 68.7), turned to 270 degrees
- moved C16 40.1 mm to (62.6, 66.4), turned to 180 degrees
- moved R7 40.0 mm to (62.9, 104.8)
- moved R9 40.0 mm to (62.9, 112.9)
- moved R4 39.8 mm to (90.0, 131.1)
- moved JP1 39.8 mm to (63.2, 107.4)
- moved C10 38.8 mm to (62.6, 63.5), turned to 180 degrees
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Connections:
- net Net-(C6-Pad2) renamed /+
- net Net-(C7-Pad2) renamed /-
- net Net-(RV1-Pad1) renamed /mono
Routing:
- net +BATT: track 0.00 -> 29.7 mm
- net Net-(JP6-Pad2): track 0.00 -> 8.32 mm
- net Net-(C16-Pad2): track 0.00 -> 4.15 mm
- net Net-(JP5-Pad2): track 0.00 -> 3.75 mm
- net GND: track 0.00 -> 3.08 mm
- net Net-(C16-Pad1): track 0.00 -> 2.44 mm
- net Net-(C9-Pad1): track 0.00 -> 2.35 mm
- net Net-(C7-Pad1): track 0.00 -> 2.35 mm
- net Net-(C10-Pad1): track 0.00 -> 2.34 mm
- net Net-(C8-Pad1): track 0.00 -> 1.92 mm
- net Net-(C6-Pad1): track 0.00 -> 1.92 mm
Other:
- outline, holes or cut-outs redrawn

Commit message: work in progress
Parts:
- removed the C5 at (74.0, 100.2)
- removed the D2 at (95.4, 126.6)
- removed D4, D5: LED, LED_SMD:LED_0603_1608Metric
- removed the JP2 at (51.2, 103.0)
- removed the JP3 at (58.7, 107.8)
- removed JP7: Jumper_NC_Dual, Connector_PinHeader_2.54mm:PinHeader_1x03_P2.54mm_Vertical
- removed the R1 at (92.2, 128.2)
- added C24: 1uF, Capacitor_SMD:C_0603_1608Metric, F.Cu at (79.9, 116.3)
- added J6: Conn_01x06, Connector_PinHeader_2.54mm:PinHeader_2x03_P2.54mm_Vertical, F.Cu at (96.6, 105.0)
- added Q1: AO3400, Package_TO_SOT_SMD:SOT-23, F.Cu at (79.6, 96.6)
- added Q2: AO3400, Package_TO_SOT_SMD:SOT-23, F.Cu at (79.4, 112.5)
- added Q3: AO3401, Package_TO_SOT_SMD:SOT-23, F.Cu at (86.4, 92.2)
- added R10: 10k, Resistor_SMD:R_0603_1608Metric, F.Cu at (75.2, 96.6)
- added R13: 10k, Resistor_SMD:R_0603_1608Metric, F.Cu at (78.4, 111.3)
- added R14: 10k, Resistor_SMD:R_0603_1608Metric, F.Cu at (78.4, 113.8)
- added R15: 1k, Resistor_SMD:R_0603_1608Metric, F.Cu at (92.7, 88.5)
- added R16: 10k, Resistor_SMD:R_0603_1608Metric, F.Cu at (92.7, 91.0)
- added R20: 10k, Resistor_SMD:R_0603_1608Metric, F.Cu at (82.8, 108.0)
- added R21: 1k, Resistor_SMD:R_0603_1608Metric, F.Cu at (103.6, 96.8)
- added R22: 1k, Resistor_SMD:R_0603_1608Metric, F.Cu at (103.6, 98.3)
- added R23: 1k, Resistor_SMD:R_0603_1608Metric, F.Cu at (103.6, 99.8)
- added R24: 1k, Resistor_SMD:R_0603_1608Metric, F.Cu at (103.6, 101.3)
- added R9: 1k, Resistor_SMD:R_0603_1608Metric, F.Cu at (76.8, 96.6)
- C3: value 100u -> 10u; footprint Capacitor_SMD:CP_Elec_6.3x7.7 -> Capacitor_SMD:C_0603_1608Metric
- D1: value STDBY -> BAT54C; footprint LED_SMD:LED_0603_1608Metric -> Package_TO_SOT_SMD:SOT-23
- R1: renamed from R2; value 1k -> 10k
- R11: value 1k -> 10k
- R19: renamed from R10; value 100 -> 1k
- R7: renamed from R8; value 1k -> 10k
- R8: renamed from R9; value 1k -> 10k
- U7: value CAT809 -> ATtiny13A; footprint Package_TO_SOT_SMD:SOT-23 -> Package_SO:SOIC-8_3.9x4.9mm_P1.27mm
- moved C22 29.4 mm to (107.6, 72.8)
- moved R7 25.5 mm to (70.6, 95.8)
- moved R12 19.9 mm to (72.8, 118.7)
- moved D1 18.3 mm to (86.4, 112.3), turned to 180 degrees
- moved R11 18.2 mm to (84.5, 103.8)
- moved R8 16.1 mm to (70.6, 98.8), turned to 0 degrees
- moved U7 15.2 mm to (94.2, 99.9)
- moved R2 14.7 mm to (81.5, 126.2), turned to 180 degrees
- moved RV3 14.1 mm to (92.5, 64.3), turned to 90 degrees
- moved C4 12.4 mm to (70.6, 94.2)
- moved C23 11.5 mm to (96.8, 95.2), turned to 90 degrees
- moved R3 10.6 mm to (81.5, 124.7)
- moved RV2 10.5 mm to (98.9, 64.3), turned to 90 degrees
- moved C3 9.66 mm to (70.6, 97.3)
- moved R19 9.65 mm to (84.2, 75.4), turned to 90 degrees
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- renumbered C16 to C10, C17 to C16, C18 to C17, C19 to C18, C20 to C19, C21 to C20, C22 to C21, C23 to C22, C24 to C23, C6 to C5, C7 to C6, C8 to C7, C9 to C8, C10 to C9, D3 to D2, JP4 to JP2, JP5 to JP3, JP6 to JP4, R13 to R17, R14 to R18, R3 to R2, R4 to R3, R5 to R4, R6 to R5, R7 to R6
Connections:
- C23 pad 1: +BATT -> VCC
- D1 pad 1: Net-(D1-Pad1) -> VBUS
- D1 pad 2: VBUS -> +BATT
- D2 pad 1: Net-(D3-Pad1) -> GND
- J1 pad S1: GND -> Net-(J1-PadS1)
- R1 pad 1: Net-(D2-Pad1) -> VBUS
- R1 pad 2: Net-(R2-Pad2) (its old number) -> CHRG
- R11 pad 1: Net-(D4-Pad1) -> VCC
- R11 pad 2: Net-(R11-Pad2) -> Blue
- R12 pad 2: Net-(R12-Pad2) -> MUTE
- R19 pad 1: +BATT -> Net-(R19-Pad1)
- U1 pad 7: Net-(R2-Pad2) (its old number) -> CHRG
- U4 pad 1: LED -> Net-(R9-Pad2)
- U4 pad 2: Net-(R12-Pad2) -> Net-(U4-Pad2)
- U4 pad 3: Net-(R11-Pad2) -> Net-(U4-Pad3)
- U6 pad 1: Net-(J4-Pad2) -> Net-(J4-Pad1)
- U6 pad 3: Net-(J4-Pad1) -> Net-(J4-Pad2)
- U7 pad 1: GND -> Net-(J6-Pad5)
- U7 pad 2: Net-(JP7-Pad1) -> Blue
- U7 pad 3: +BATT -> Net-(R19-Pad1)
Routing:
- net +BATT: track 29.7 -> 162.2 mm, vias 0 -> 3
- net Net-(F1-Pad1): track 0.00 -> 111.8 mm, vias 0 -> 1
- net /-: track 0.00 -> 30.0 mm
- net /+: track 0.00 -> 29.3 mm
- net Net-(R9-Pad2): track 0.00 -> 25.7 mm, vias 0 -> 2
- net VBUS: track 0.00 -> 23.9 mm
- net MOSI: track 0.00 -> 21.9 mm
- net Net-(RV1-Pad2): track 0.00 -> 19.9 mm
- net Net-(C2-Pad2): track 0.00 -> 19.6 mm
- net CLK: track 0.00 -> 18.9 mm
- net Net-(J5-Pad2): track 0.00 -> 17.1 mm
- net /mono: track 0.00 -> 16.9 mm
- net VCC: track 0.00 -> 16.8 mm
- net CSB: track 0.00 -> 15.9 mm
- net MISO: track 0.00 -> 13.0 mm
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- added copper zone on F.Cu, net +BATT
Other:
- outline, holes or cut-outs redrawn
- board text added: "CLK"
- board text added: "CSB"
- board text added: "GND"
- board text added: "MISO"
- board text added: "MOSI"
